Commit message: modified:   grandslam_description/urdf/grandslam.xacro 	modified:   robot_localization/params/ekf.yaml 	modified:   slam_gmapping/slam_gmapping/src/slam_gmapping.cpp 	deleted:    tf_to_odom/CMakeLists.txt 	deleted:    tf_to_odom/launch/tf_to_odom_launch.py 	deleted:    tf_to_odom/package.xml 	deleted:    tf_to_odom/setup.py 	new file:   tf_to_topic/launch/tf_to_topic.launch.py 	new file:   tf_to_topic/package.xml 	renamed:    tf_to_odom/tf_to_odom/__init__.py -> tf_to_topic/resource/tf_to_topic 	new file:   tf_to_topic/setup.cfg 	new file:   tf_to_topic/setup.py 	new file:   tf_to_topic/test/test_copyright.py 	new file:   tf_to_topic/test/test_flake8.py 	new file:   tf_to_topic/test/test_pep257.py 	new file:   tf_to_topic/tf_to_topic/__init__.py 	new file:   tf_to_topic/tf_to_topic/__pycache__/__init__.cpython-38.pyc 	new file:   tf_to_topic/tf_to_topic/__pycache__/tf_to_topic_node.cpython-38.pyc 	renamed:    tf_to_odom/tf_to_odom/tf_to_odom_node.py -> tf_to_topic/tf_to_topic/tf_to_topic_node.py

File: grandslam_description/urdf/grandslam.xacro (robot description, xacro)
@@ -14,21 +14,16 @@
         <color rgba="0 0 1 1" />
     </material>
-  <!-- Base -->
-  <link name = "base_link">
+  <!-- Base_footprint -->
+  <link name = "base_footprint">
   </link>
-  <!--odom LINK-->
-  <joint name="odom_link" type="fixed">
-    <parent link="odom"/>
-    <child link ="base_link"/>
-  </joint>
-  <!-- BODY LINK -->
-  <joint name="body_joint" type="fixed">
-    <parent link="base_link"/>
-    <child link="body"/>
+  <!-- base_link LINK -->
+  <joint name="base_link_joint" type="fixed">
+    <parent link="base_footprint"/>
+    <child link="base_link"/>
   </joint>
   <!--sensor_box LINK-->
   <joint name="sensor_box_link" type="fixed">
     <origin xyz="0.0 -0.1 0.335" rpy="0.0 0.0 0.0"/>
-    <parent link="body"/>
+    <parent link="base_link"/>
     <child link ="sensor_box"/>
   </joint>
@@ -44,6 +39,6 @@
     <child link ="imu"/>
   </joint>
-  <!-- Body -->
-  <link name="body">
+  <!-- base_link -->
+  <link name="base_link">
     <visual>
       <geometry>
@@ -74,6 +69,3 @@
   <link name="imu">
   </link>
-  <!--odom-->
-  <link name="odom">
-  </link>
 </robot>

Commit message: new file:   convert_encoder/convert_encoder/__init__.py 	new file:   convert_encoder/convert_encoder/speed_estimator.py 	new file:   convert_encoder/launch/speed_estimator_launch.py 	new file:   convert_encoder/package.xml 	new file:   convert_encoder/resource/convert_encoder 	new file:   convert_encoder/setup.cfg 	new file:   convert_encoder/setup.py 	new file:   convert_encoder/test/test_copyright.py 	new file:   convert_encoder/test/test_flake8.py 	new file:   convert_encoder/test/test_pep257.py 	modified:   grandslam_description/urdf/grandslam.xacro 	modified:   robot_localization/params/ekf.yaml

File: grandslam_description/urdf/grandslam.xacro (robot description, xacro)
@@ -24,5 +24,5 @@
   <!--sensor_box LINK-->
   <joint name="sensor_box_link" type="fixed">
-    <origin xyz="0.0 -0.1 0.335" rpy="0.0 0.0 0.0"/>
+    <origin xyz="-0.1 0.0 0.335" rpy="0.0 0.0 0.0"/>
     <parent link="base_link"/>
     <child link ="sensor_box"/>
@@ -43,5 +43,5 @@
     <visual>
       <geometry>
-        <box size="0.75 1.30 0.47"/>
+        <box size="1.30 0.75 0.47"/>
       </geometry>
       <material name="blue"/>
@@ -52,5 +52,5 @@
     <visual>
       <geometry>
-        <box size="0.4 0.3 0.2"/>
+        <box size="0.3 0.4 0.2"/>
       </geometry>
       <material name="green"/>
